Commit message: quick fix urdf

File: urdf/kortex_dual_robots.urdf (robot description, URDF)
Before this commit: robot dual_robot, 27 links, 26 joints
Links:
- link left_base_link: geometry collision mesh filename=package://meshes/base_link.STL; visual mesh filename=package://meshes/base_link.STL
- link left_bracelet_link: geometry collision mesh filename=package://meshes/bracelet_with_vision_link.STL; visual mesh filename=package://meshes/bracelet_with_vision_link.STL
- link left_forearm_link: geometry collision mesh filename=package://meshes/forearm_link.STL; visual mesh filename=package://meshes/forearm_link.STL
- link left_half_arm_1_link: geometry collision mesh filename=package://meshes/half_arm_1_link.STL; visual mesh filename=package://meshes/half_arm_1_link.STL
- link left_half_arm_2_link: geometry collision mesh filename=package://meshes/half_arm_2_link.STL; visual mesh filename=package://meshes/half_arm_2_link.STL
- link left_shoulder_link: geometry collision mesh filename=package://meshes/shoulder_link.STL; visual mesh filename=package://meshes/shoulder_link.STL
- link left_spherical_wrist_1_link: geometry collision mesh filename=package://meshes/spherical_wrist_1_link.STL; visual mesh filename=package://meshes/spherical_wrist_1_link.STL
- link left_spherical_wrist_2_link: geometry collision mesh filename=package://meshes/spherical_wrist_2_link.STL; visual mesh filename=package://meshes/spherical_wrist_2_link.STL
- link right_base_link: geometry collision mesh filename=package://meshes/base_link.STL; visual mesh filename=package://meshes/base_link.STL
- link right_bracelet_link: geometry collision mesh filename=package://meshes/bracelet_with_vision_link.STL; visual mesh filename=package://meshes/bracelet_with_vision_link.STL
- link right_forearm_link: geometry collision mesh filename=package://meshes/forearm_link.STL; visual mesh filename=package://meshes/forearm_link.STL
- link right_half_arm_1_link: geometry collision mesh filename=package://meshes/half_arm_1_link.STL; visual mesh filename=package://meshes/half_arm_1_link.STL
- link right_half_arm_2_link: geometry collision mesh filename=package://meshes/half_arm_2_link.STL; visual mesh filename=package://meshes/half_arm_2_link.STL
- link right_shoulder_link: geometry collision mesh filename=package://meshes/shoulder_link.STL; visual mesh filename=package://meshes/shoulder_link.STL
- link right_spherical_wrist_1_link: geometry collision mesh filename=package://meshes/spherical_wrist_1_link.STL; visual mesh filename=package://meshes/spherical_wrist_1_link.STL
- link right_spherical_wrist_2_link: geometry collision mesh filename=package://meshes/spherical_wrist_2_link.STL; visual mesh filename=package://meshes/spherical_wrist_2_link.STL
